Commit message: Fix(farol_vehicles): cofigurarions for bluerov, heavy and regular configurations and correct gazebo launch file

File: farol_vehicles/bluerov_heavy_vehicle/robots/default.xacro (robot description, xacro)
@@ -5,6 +5,6 @@
   <xacro:arg name="inertial_reference_frame" default="world"/>
   <!-- Include the ROV macro file -->
-  <xacro:include filename="$(find bluerov_regular)/urdf/base.xacro"/>
-  <xacro:include filename="$(find bluerov_regular)/urdf/gazebo.xacro"/>
+  <xacro:include filename="$(find bluerov_heavy_vehicle)/urdf/base.xacro"/>
+  <xacro:include filename="$(find bluerov_heavy_vehicle)/urdf/gazebo.xacro"/>
   <!-- Create the bluerov -->
   <xacro:bluerov_base

File: farol_vehicles/bluerov_heavy_vehicle/urdf/base.xacro (robot description, xacro)
@@ -8,5 +8,5 @@
   <xacro:include filename="$(find uuv_gazebo_ros_plugins)/urdf/snippets.xacro"/>
     <!-- Loading vehicle's specific macros -->
-  <xacro:include filename="$(find bluerov_heavy)/urdf/snippets.xacro"/>
+  <xacro:include filename="$(find bluerov_heavy_vehicle)/urdf/snippets.xacro"/>
     <!--
       Vehicle's parameters (remember to enter the model parameters below)
@@ -32,9 +32,9 @@
       Open the meshes for the RexROV vehicle in Blender to see an example on the mesh placement.
     -->
-      <xacro:property name="visual_mesh_file" value="file://$(find bluerov_heavy)/meshes/bluerov_noprop.dae"/>
+      <xacro:property name="visual_mesh_file" value="file://$(find bluerov_heavy_vehicle)/meshes/bluerov_noprop.dae"/>
         <!-- Collision geometry mesh, usually in STL format (it is recommended to keep
           this geometry as simple as possible to improve the performance the physics engine
         regarding the computation of collision forces) -->
-      <xacro:property name="collision_mesh_file" value="file://$(find bluerov_heavy)/meshes/bluerov_noprop.stl"/>
+      <xacro:property name="collision_mesh_file" value="file://$(find bluerov_heavy_vehicle)/meshes/bluerov_noprop.stl"/>
         <!-- Vehicle macro -->
       <xacro:macro name="bluerov_base" params="namespace *gazebo inertial_reference_frame">
@@ -73,7 +73,7 @@
         <xacro:insert_block name="gazebo"/>
             <!-- Include the thruster modules -->
-            <xacro:include filename="$(find bluerov_heavy)/urdf/actuators.xacro"/>
+            <xacro:include filename="$(find bluerov_heavy_vehicle)/urdf/actuators.xacro"/>
             <!-- Include the sensor modules -->
-            <xacro:include filename="$(find bluerov_heavy)/urdf/sensors.xacro"/>
+            <xacro:include filename="$(find bluerov_heavy_vehicle)/urdf/sensors.xacro"/>
         </xacro:macro>
 </robot>

File: farol_vehicles/bluerov_heavy_vehicle/urdf/snippets.xacro (robot description, xacro)
@@ -7,5 +7,5 @@
   over propeller's frame X-axis in DAE (Collada) or STL format.
   -->
-  <xacro:property name="prop_mesh_file" value="file://$(find bluerov_regular)/meshes/bluerov_propcw.dae"/>
+  <xacro:property name="prop_mesh_file" value="file://$(find bluerov_heavy_vehicle)/meshes/bluerov_propcw.dae"/>
   <!--
     Thruster macro with integration of joint and link. The thrusters should

File: farol_vehicles/bluerov_regular_vehicle/robots/default.xacro (robot description, xacro)
@@ -5,6 +5,6 @@
   <xacro:arg name="inertial_reference_frame" default="world"/>
   <!-- Include the ROV macro file -->
-  <xacro:include filename="$(find bluerov_heavy)/urdf/base.xacro"/>
-  <xacro:include filename="$(find bluerov_heavy)/urdf/gazebo.xacro"/>
+  <xacro:include filename="$(find bluerov_regular_vehicle)/urdf/base.xacro"/>
+  <xacro:include filename="$(find bluerov_regular_vehicle)/urdf/gazebo.xacro"/>
   <!-- Create the bluerov -->
   <xacro:bluerov_base

File: farol_vehicles/bluerov_regular_vehicle/urdf/base.xacro (robot description, xacro)
@@ -8,5 +8,5 @@
   <xacro:include filename="$(find uuv_gazebo_ros_plugins)/urdf/snippets.xacro"/>
     <!-- Loading vehicle's specific macros -->
-  <xacro:include filename="$(find bluerov_regular)/urdf/snippets.xacro"/>
+  <xacro:include filename="$(find bluerov_regular_vehicle)/urdf/snippets.xacro"/>
     <!--
       Vehicle's parameters (remember to enter the model parameters below)
@@ -30,9 +30,9 @@
       Open the meshes for the RexROV vehicle in Blender to see an example on the mesh placement.
     -->
-      <xacro:property name="visual_mesh_file" value="file://$(find bluerov_regular)/meshes/bluerov_noprop.dae"/>
+      <xacro:property name="visual_mesh_file" value="file://$(find bluerov_regular_vehicle)/meshes/bluerov_noprop.dae"/>
         <!-- Collision geometry mesh, usually in STL format (it is recommended to keep
           this geometry as simple as possible to improve the performance the physics engine
         regarding the computation of collision forces) -->
-      <xacro:property name="collision_mesh_file" value="file://$(find bluerov_regular)/meshes/bluerov_noprop.stl"/>
+      <xacro:property name="collision_mesh_file" value="file://$(find bluerov_regular_vehicle)/meshes/bluerov_noprop.stl"/>
         <!-- Vehicle macro -->
       <xacro:macro name="bluerov_base" params="namespace *gazebo inertial_reference_frame">
@@ -67,7 +67,7 @@
         <xacro:insert_block name="gazebo"/>
             <!-- Include the thruster modules -->
-            <xacro:include filename="$(find bluerov_regular)/urdf/actuators.xacro"/>
+            <xacro:include filename="$(find bluerov_regular_vehicle)/urdf/actuators.xacro"/>
             <!-- Include the sensor modules -->
-            <xacro:include filename="$(find bluerov_regular)/urdf/sensors.xacro"/>
+            <xacro:include filename="$(find bluerov_regular_vehicle)/urdf/sensors.xacro"/>
         </xacro:macro>
 </robot>

File: farol_vehicles/bluerov_regular_vehicle/urdf/snippets.xacro (robot description, xacro)
@@ -7,5 +7,5 @@
   over propeller's frame X-axis in DAE (Collada) or STL format.
   -->
-  <xacro:property name="prop_mesh_file" value="file://$(find bluerov_heavy)/meshes/bluerov_propcw.dae"/>
+  <xacro:property name="prop_mesh_file" value="file://$(find bluerov_regular_vehicle)/meshes/bluerov_propcw.dae"/>
   <!--
     Thruster macro with integration of joint and link. The thrusters should
