Commit message: Update(farol_vehicles): Changed vehicle name from mvector to myellow and deleted the previous myellow vehicle

File: farol_vehicles/myellow_vehicle/robots/default.xacro (robot description, xacro)
@@ -1,4 +1,5 @@
 <?xml version="1.0"?>
 <robot name="myellow" xmlns:xacro="http://www.ros.org/wiki/xacro" >
+  <!-- Initial parameters -->
   <xacro:arg name="debug" default="0"/>
   <xacro:arg name="namespace" default="myellow"/>

File: farol_vehicles/myellow_vehicle/urdf/actuators.xacro (robot description, xacro)
@@ -8,22 +8,30 @@
     aware that Gazebo does not use the SNAME convention per default.
   -->
-      <!--left horizontal thruster-->
+    <!--left horizontal back thruster-->
     <xacro:thruster_macro robot_namespace="${namespace}" thruster_id="0">
-      <origin xyz="-0.290 0.14 0.011" rpy="0 0 0" />
+      <origin xyz="-0.306 0.062 0.0" rpy="0 0 ${0.25*pi}" />
     </xacro:thruster_macro>
-    <!--right horizontal thruster-->
+    <!--right horizontal back thruster-->
     <xacro:thruster_macro robot_namespace="${namespace}" thruster_id="1">
-      <origin xyz="-0.290 -0.140 0.011" rpy="0 0 0" />
+      <origin xyz="-0.306 -0.062 0.0" rpy="0 0 -${0.25*pi}" />
     </xacro:thruster_macro>
-    <!--left vertical thruster-->
+     <!--left vertical thruster-->
     <xacro:thruster_macro robot_namespace="${namespace}" thruster_id="2">
-      <origin xyz="-0.012 -0.140 -0.107" rpy="0 -${0.5*pi} 0" />
+      <origin xyz="0.087 -0.120 -0.12" rpy="0 -${0.5*pi} 0" />
     </xacro:thruster_macro>
     <!--right vertical thruster-->
     <xacro:thruster_macro robot_namespace="${namespace}" thruster_id="3">
-      <origin xyz="-0.012 0.140 -0.107" rpy="0 -${0.5*pi} 0" />
+      <origin xyz="0.087 0.120 -0.12" rpy="0 -${0.5*pi} 0" />
+    </xacro:thruster_macro>
+   <!--left horizontal front thruster-->
+    <xacro:thruster_macro robot_namespace="${namespace}" thruster_id="4">
+      <origin xyz="0.300 0.197 0.0" rpy="0 0 -${0.25*pi}" />
+    </xacro:thruster_macro>
+    <!--right horizontal front thruster-->
+    <xacro:thruster_macro robot_namespace="${namespace}" thruster_id="5">
+      <origin xyz="0.300 -0.197 0.0" rpy="0 0 ${0.25*pi}" />
     </xacro:thruster_macro>
     <!-- Thruster manager plugin to translate DSOR stack thruster msgs towards the UUV simulator -->
-    <xacro:thruster_manager_macro robot_namespace="${namespace}" number_thrusters="4" dsor_topic_thrusters="/${namespace}/thrusters/rpm_command">
+    <xacro:thruster_manager_macro robot_namespace="${namespace}" number_thrusters="6" dsor_topic_thrusters="/${namespace}/thrusters/rpm_command">
     </xacro:thruster_manager_macro>
   </robot>

File: farol_vehicles/myellow_vehicle/urdf/gazebo.xacro (robot description, xacro)
@@ -16,5 +16,5 @@
           <width>0.350</width>
           <length>1.035</length>
-          <height>0.875</height>
+          <height>0.450</height>
         </box>
         <center_of_buoyancy>${myellow_cob}</center_of_buoyancy>
@@ -31,11 +31,7 @@
           </added_mass>
           <!-- Linear damping: see p.31 in Berg2012 -->
-          <linear_damping>
-           -0.2 -55.1 -4.1879 -3000.0 -3000.0 -4.14
-          </linear_damping>
+          <linear_damping>-0.2 -55.1 -4.1879 -3000.0 -3000.0 -4.14</linear_damping>
           <!-- Non-linear damping: see p.30 in Berg2012 -->
-          <quadratic_damping>
-           -25 -101.3 -40.9649  -3000.0 -3000.0 -6.23
-          </quadratic_damping>
+          <quadratic_damping>-25 -101.3 -40.9649  -3000.0 -3000.0 -6.23</quadratic_damping>
         </hydrodynamic_model>
       </link>

File: farol_vehicles/myellow_vehicle/urdf/sensors.xacro (robot description, xacro)
@@ -32,4 +32,10 @@
     <origin xyz="-0.3 0 -0.265" rpy="0 ${0.5*pi} 0"/>
   </xacro:farol_altimeter>
+  <!-- Multibeam  -->
+  <!--xacro:forward_multibeam_p900
+    namespace="${namespace}"
+    parent_link="${namespace}/base_link">
+    <origin xyz="0.37 0 -0.32" rpy="0 ${0.5*pi} 0"/>
+  </xacro:forward_multibeam_p900-->
   <!-- RPT  -->
   <!--<xacro:default_rpt namespace="${namespace}" parent_link="${namespace}/base_link">-->
@@ -40,3 +46,7 @@
     <origin xyz="0 0 0" rpy="0 0 0"/>
   </xacro:default_pressure>
+  <!-- Mount a camera  -->
+  <!-- <xacro:default_camera namespace="${namespace}" parent_link="${namespace}/base_link" suffix="">
+    <origin xyz="0 0 -0.265" rpy="0 1.57 0"/>
+  </xacro:default_camera> -->
 </robot>

File: farol_vehicles/myellow_vehicle/urdf/snippets.xacro (robot description, xacro)
@@ -57,8 +57,5 @@
         <thrustMin>-36</thrustMin>
         <thrustMax>36</thrustMax>
-        <!--
-        Value from 0 to 1 to set the efficiency of the output thrust force
-        Default value is 1.0
-        -->
+        <!-- Value from 0 to 1 to set the efficiency of the output thrust force. Default value is 1.0 -->
         <thrust_efficiency>1</thrust_efficiency>
         <propeller_efficiency>1</propeller_efficiency>
@@ -68,12 +65,5 @@
           <timeConstant>0.346</timeConstant>
         </dynamics>
-        <!-- 2) Dead-zone nonlinearity described in Bessa, 2006
-        Input: x
-        Output: thrust
-        Function:
-        thrust = rotorConstantL * (x * abs(x) - deltaL), if x * abs(x) <= deltaL
-        thrust = 0, if deltaL < x * abs(x) < deltaR
-        thrust = rotorConstantR * (x * abs(x) - deltaR), if x * abs(x) >= deltaL
-        -->
+        <!-- Thrust curve conversion -->
         <conversion>
           <type>Bessa</type>
@@ -85,4 +75,5 @@
       </plugin>
     </gazebo>
+    <!-- Make the thruster not be affected by collisions with other object -->
     <gazebo reference="${robot_namespace}/thruster_${thruster_id}">
       <selfCollide>false</selfCollide>
@@ -99,120 +90,3 @@
     </gazebo>
   </xacro:macro>
-  <xacro:macro name="blueview_p900_gpu"
-  params="namespace parent_link suffix camera_name mass *inertia *origin update_rate horizontal_fov vertical_fov_pixels max_distance min_distance ray_skips plot_scaler debug scale">
-    <xacro:forward_looking_sonar_gpu
-      namespace="${namespace}"
-      parent_link="${parent_link}"
-      suffix="${suffix}"
-      mass="${mass}"
-      camera_name="${camera_name}"
-      update_rate="${update_rate}"
-      horizontal_fov="${horizontal_fov}"
-      vertical_fov_pixels="${vertical_fov_pixels}"
-      max_distance="${max_distance}"
-      min_distance="${min_distance}"
-      ray_skips="${ray_skips}"
-      plot_scaler="${plot_scaler}"
-      debug="${debug}"
-      scale="${scale}"
-      sonar_freq="900e3"
-      bandwidth="29.9e3"
-      sound_speed="1500"
-      source_level="220"
-      sensor_gain="0.2">
-      <xacro:insert_block name="inertia" />
-      <xacro:insert_block name="origin" />
-    </xacro:forward_looking_sonar_gpu>
-  </xacro:macro>
-  <xacro:macro name="forward_looking_sonar_gpu"
-    params="namespace parent_link suffix camera_name mass *inertia *origin update_rate horizontal_fov vertical_fov_pixels max_distance min_distance ray_skips plot_scaler debug scale sonar_freq bandwidth sound_speed source_level sensor_gain">
-    <!-- Sensor link -->
-    <link name="${namespace}/forward_sonar${suffix}_link">
-      <inertial>
-        <xacro:insert_block name="inertia" />
-        <mass value="${mass}" />
-        <origin xyz="0 0 0" rpy="0 0 0"/>
-      </inertial>
-      <visual>
-        <geometry>
-          <mesh filename="file://$(find uuv_sensor_ros_plugins)/meshes/p900.dae" scale="${scale}"/>
-        </geometry>
-      </visual>
-      <xacro:no_collision/>
-    </link>
-    <joint name="${namespace}_forward_sonar${suffix}_joint" type="revolute">
-      <xacro:insert_block name="origin" />
-      <parent link="${parent_link}" />
-      <child link="${namespace}/forward_sonar${suffix}_link" />
-      <limit upper="0" lower="0" effort="0" velocity="0" />
-      <axis xyz="1 0 0"/>
-    </joint>
-    <gazebo reference="${namespace}/forward_sonar${suffix}_link">
-      <sensor name="${namespace}/image_sonar" type="depth">
-        <parent link="${namespace}/forward_sonar_link"/>
-        <xacro:insert_block name="origin" />
-        <visualize>true</visualize>
-        <always_on>true</always_on>
-        <update_rate>${update_rate}</update_rate>
-        <camera>
-          <!-- 90 degrees for the M900-90 -->
-          <!-- <horizontal_fov>1.57079632679</horizontal_fov> -->
-          <!-- 130 degrees for the P900-130 -->
-          <horizontal_fov>${horizontal_fov}</horizontal_fov>
-          <image>
-            <width>512</width>
-            <!-- Set vertical FOV by setting image height -->
-            <!-- For 20 deg. -->
-            <height>${vertical_fov_pixels}</height>
-            <format>R8G8B8</format>
-          </image>
-          <clip>
-            <near>0.1</near>
-            <far>1000</far>
-          </clip>
-          <depth_camera>
-            <output>depths</output>
-          </depth_camera>
-          <save enabled="false">
-            <path>/tmp/camera</path>
-          </save>
-        </camera>
-        <plugin filename="libnps_multibeam_sonar_ros_plugin.so" name="${namespace}_forward_sonar">
-          <!-- Sonar properties -->
-          <sonarFreq>${sonar_freq}</sonarFreq>
-          <bandwidth>${bandwidth}</bandwidth>
-          <soundSpeed>${sound_speed}</soundSpeed>
-          <sourceLevel>${source_level}</sourceLevel>
-          <maxDistance>${max_distance}</maxDistance>
-          <minDistance>${min_distance}</minDistance>
-          <constantReflectivity>true</constantReflectivity>
-          <!-- The CSV databsefile is located at the worlds folder -->
-          <reflectivityDatabaseFile>variationalReflectivityDatabase.csv</reflectivityDatabaseFile>
-          <raySkips>${ray_skips}</raySkips>
-          <sensorGain>${sensor_gain}</sensorGain>
-          <plotScaler>${plot_scaler}</plotScaler>
-          <writeLog>false</writeLog>
-          <debugFlag>${debug}</debugFlag>
-          <writeFrameInterval>5</writeFrameInterval>
-          <!-- This name is prepended to ROS topics -->
-          <cameraName>${camera_name}</cameraName>
-          <!-- ROS publication topics -->
-          <imageTopicName>image_raw</imageTopicName>
-          <cameraInfoTopicName>image_raw/camera_info</cameraInfoTopicName>
-          <pointCloudTopicName>point_cloud</pointCloudTopicName>
-          <depthImageTopicName>image_depth</depthImageTopicName>
-          <depthImageCameraInfoTopicName>image_depth/camera_info</depthImageCameraInfoTopicName>
-          <sonarImageRawTopicName>sonar_image_raw</sonarImageRawTopicName>
-          <sonarImageTopicName>sonar_image</sonarImageTopicName>
-          <frameName>forward_sonar_optical_link</frameName>
-        </plugin>
-      </sensor>
-    </gazebo>
-    <joint name="${namespace}/forward_sonar${suffix}_joint" type="fixed">
-        <origin xyz="0 0 0" rpy="0 0 0"/>
-        <parent link="${namespace}/forward_sonar${suffix}_link"/>
-        <child link="${namespace}/forward_sonar${suffix}_optical_frame"/>
-      </joint>
-  	<link name="${namespace}/forward_sonar${suffix}_optical_frame"/>
-  </xacro:macro>
 </robot>
