Commit message: Update(farol_vehicles): changed dvl and altimeter position on myellow to match the real vehicle

File: farol_vehicles/myellow_vehicle/urdf/sensors.xacro (robot description, xacro)
@@ -19,5 +19,5 @@
     parent_link="${namespace}/base_link"
     inertial_reference_frame="${inertial_reference_frame}">
-    <origin xyz="-0.5 0 -0.265" rpy="0 ${0.5*pi} 0"/>
+    <origin xyz="0.45 0 -0.2" rpy="0 ${0.5*pi} 0"/>
   </xacro:default_dvl_macro>
   <!-- IMU  -->
@@ -30,5 +30,5 @@
   <!-- Altimeter sensor -->
   <xacro:farol_altimeter namespace="${namespace}" parent_link="$(arg namespace)/base_link" suffix="">
-    <origin xyz="-0.3 0 -0.265" rpy="0 ${0.5*pi} 0"/>
+    <origin xyz="-0.35 0 -0.25" rpy="0 ${0.5*pi} 0"/>
   </xacro:farol_altimeter>
   <!-- Multibeam  -->
