Commit message: incomplete push -> moving to sturgeon

File: farol_vehicles/myellow_vehicle/urdf/base.xacro (robot description, xacro)
@@ -12,7 +12,7 @@
       Vehicle's parameters (remember to enter the model parameters below)
     -->
-  <xacro:property name="mass" value="28.5"/>
+  <xacro:property name="mass" value="29.32"/>
     <!-- Center of gravity -->
-  <xacro:property name="cog" value="0 0 0"/>
+  <xacro:property name="cog" value="0 0 -0.1"/>
     <!-- Fluid density -->
   <xacro:property name="rho" value="1028"/>
@@ -40,6 +40,6 @@
             <mass value="${mass}" />
             <origin xyz="${cog}" rpy="0 0 0"/>
-            <inertia ixx="1000" ixy="0" ixz="0"
-            iyy="1000" iyz="0"
+            <inertia ixx="100000" ixy="0" ixz="0"
+            iyy="100000" iyz="0"
             izz="4.14" />
           </inertial>

File: farol_vehicles/myellow_vehicle/urdf/gazebo.xacro (robot description, xacro)
@@ -2,8 +2,8 @@
 <robot xmlns:xacro="http://www.ros.org/wiki/xacro">
     <!-- Center of buoyancy -->
-    <xacro:property name="myellow_cob" value="0 0 0"/>
+    <xacro:property name="myellow_cob" value="0 0 0.01"/>
     <!-- Vehicle's actual volume (Gazebo cannot compute the volume out of the mesh) -->
     <xacro:property name="myellow_volume" value="0.0287309120146"/>
-    <!--<xacro:property name="myellow_volume" value="0.034582136"/>-->
+    <!-- <xacro:property name="myellow_volume" value="0.034582136"/> -->
     <xacro:macro name="myellow_hydro_model" params="namespace">
       <!-- List of hydrodynamic models this robot's links -->
@@ -26,12 +26,12 @@
             0     30    0     0     0     0
             0     0     70    0     0     0
-            0     0     0     0     0     0
-            0     0     0     0     0     0
-            0     0     0     0     0     .5
+            0     0     0     100000   0     0
+            0     0     0     0     100000     0
+            0     0     0     0     0     0.5
           </added_mass>
           <!-- Linear damping: see p.31 in Berg2012 -->
-          <linear_damping>-0.2 -55.1 -4.1879 -3000.0 -3000.0 -4.14</linear_damping>
+          <linear_damping>-0.2 -55.1 -6.4369 -100000 -100000 -4.14</linear_damping>
           <!-- Non-linear damping: see p.30 in Berg2012 -->
-          <quadratic_damping>-25 -101.3 -40.9649  -3000.0 -3000.0 -6.23</quadratic_damping>
+          <quadratic_damping>-25 -101.3 -120.4854  -100000 -100000 -6.23</quadratic_damping>
         </hydrodynamic_model>
       </link>
