Commit message: Fix(mdock_vehicle): changed the orientation of mdock in order to math the correct D reference frame, which points contrary of the dock opening (x) and down (z).

File: farol_vehicles/mdock_vechicle/urdf/base.xacro (robot description, xacro)
@@ -38,5 +38,5 @@
           <inertial>
             <mass value="${mass}" />
-            <origin xyz="${cog}" rpy="0 0 0"/>
+            <origin xyz="${cog}" rpy="0 0 3.141592653589793"/>
             <inertia ixx="0" ixy="1000" ixz="1000"
             iyy="0" iyz="1000"
@@ -44,5 +44,5 @@
           </inertial>
           <visual>
-            <origin xyz="0 0 0" rpy="0 0 0"/>
+            <origin xyz="0 0 0" rpy="0 0 3.141592653589793"/>
             <geometry>
               <mesh filename="${visual_mesh_file}" scale="1 1 1" />
@@ -50,5 +50,5 @@
           </visual>
           <collision>
-            <origin xyz="0 0 0" rpy="0 0 0"/>
+            <origin xyz="0 0 0" rpy="0 0 3.141592653589793"/>
             <geometry>
               <mesh filename="${collision_mesh_file}" scale="1 1 1" />

File: farol_vehicles/mdock_vechicle/urdf/gazebo.xacro (robot description, xacro)
@@ -7,5 +7,5 @@
     <xacro:macro name="mdock_hydro_model" params="namespace">
       <!-- List of hydrodynamic models this robot's links -->
-      <link name="${namespace}/base_link">100000
+      <link name="${namespace}/base_link">
         <!-- This flag will make the link neutrally buoyant -->
         <neutrally_buoyant>0</neutrally_buoyant>
